Commit message: Added files for gazebo

File: src/basic_robotics/urdf/fwb_macros.xacro (robot description, xacro)
@@ -52,4 +52,6 @@
             - r: Radius of wheel
             - h: Height / Depth of wheel
+        Returns:
+            The <link> and <joint> elements for the wheel
     -->
     <xacro:macro name="add_wheel" params="sx sy sz lname jname m r h">

File: src/basic_robotics/urdf/fwb_parameters.xacro (robot description, xacro)
@@ -3,11 +3,11 @@
 <robot name="fw_robot" xmlns:xacro="http://www.ros.org/wiki/xacro" >
     <!-- Parameters for the robot body (cuboid) -->
-    <xacro:property name="body_m" value="2.0" />    <!-- Mass -->
-    <xacro:property name="body_sx" value="1" /> <!-- Side Length: X Axis -->
-    <xacro:property name="body_sy" value="0.5" /> <!-- Side Length: Y Axis -->
-    <xacro:property name="body_sz" value="0.25" /> <!-- Side Length: Z Axis -->
+    <xacro:property name="body_m" value="20" />    <!-- Mass (kg) -->
+    <xacro:property name="body_sx" value="0.544" /> <!-- Side Length: X Axis (m) -->
+    <xacro:property name="body_sy" value="0.420" /> <!-- Side Length: Y Axis (m) -->
+    <xacro:property name="body_sz" value="0.260" /> <!-- Side Length: Z Axis (m) -->
     <!-- Parameters for robot wheels (cylinders) -->
-    <xacro:property name="wheel_m" value="0.25" />  <!-- Mass -->
-    <xacro:property name="wheel_r" value="0.125" /> <!-- Wheel radius -->
-    <xacro:property name="wheel_h" value="0.0625" /> <!-- Wheel height -->
+    <xacro:property name="wheel_m" value="1" />  <!-- Mass (kg) -->
+    <xacro:property name="wheel_r" value="0.165" /> <!-- Wheel radius (m) -->
+    <xacro:property name="wheel_h" value="0.125" /> <!-- Wheel height (m) -->
 </robot>

File: src/basic_robotics/urdf/simple_fwb.urdf (robot description, URDF)
Before this commit: robot fw_robot, 6 links, 5 joints
Links:
- link body: mass 2.0 -> 20; geometry visual box size=0.544 0.42 0.26
- link fl_wheel: mass 0.25 -> 1; geometry visual cylinder length=0.125 radius=0.165
- link fr_wheel: mass 0.25 -> 1; geometry visual cylinder length=0.125 radius=0.165
- link hl_wheel: mass 0.25 -> 1; geometry visual cylinder length=0.125 radius=0.165
- link hr_wheel: mass 0.25 -> 1; geometry visual cylinder length=0.125 radius=0.165
Joints:
- joint body_world_fixed: origin xyz=0.0 0.0 0.25 rpy=0.0 0.0 0.0 -> xyz=0.0 0.0 0.29500000000000004 rpy=0.0 0.0 0.0
- joint fl_wheel_joint: origin xyz=0.5 0.28125 -0.125 rpy=-1.5707963267948966 0.0 0.0 -> xyz=0.272 0.27249999999999996 -0.13 rpy=-1.5707963267948966 0.0 0.0
- joint fr_wheel_joint: origin xyz=0.5 -0.28125 -0.125 rpy=-1.5707963267948966 0.0 0.0 -> xyz=0.272 -0.27249999999999996 -0.13 rpy=-1.5707963267948966 0.0 0.0
- joint hl_wheel_joint: origin xyz=-0.5 0.28125 -0.125 rpy=-1.5707963267948966 0.0 0.0 -> xyz=-0.272 0.27249999999999996 -0.13 rpy=-1.5707963267948966 0.0 0.0
- joint hr_wheel_joint: origin xyz=-0.5 0.28125 -0.125 rpy=-1.5707963267948966 0.0 0.0 -> xyz=-0.272 -0.27249999999999996 -0.13 rpy=-1.5707963267948966 0.0 0.0

File: src/basic_robotics/urdf/simple_fwb.xacro (robot description, xacro)
@@ -42,10 +42,10 @@
     <xacro:add_wheel lname="fr_wheel" jname="fr_wheel_joint"
         sx="${body_sx/2}" sy="${-(body_sy + wheel_h)/2}" sz="${-body_sz/2}"
-        m="${wheel_m}" r="${wheel_r}" h="${wheel_h}"/>  <!-- Front Left -->
+        m="${wheel_m}" r="${wheel_r}" h="${wheel_h}"/>  <!-- Front Right -->
     <xacro:add_wheel lname="hl_wheel" jname="hl_wheel_joint"
         sx="${-body_sx/2}" sy="${(body_sy + wheel_h)/2}" sz="${-body_sz/2}"
-        m="${wheel_m}" r="${wheel_r}" h="${wheel_h}"/>  <!-- Front Left -->
+        m="${wheel_m}" r="${wheel_r}" h="${wheel_h}"/>  <!-- Hind Left -->
     <xacro:add_wheel lname="hr_wheel" jname="hr_wheel_joint"
         sx="${-body_sx/2}" sy="${-(body_sy + wheel_h)/2}" sz="${-body_sz/2}"
-        m="${wheel_m}" r="${wheel_r}" h="${wheel_h}"/>  <!-- Front Left -->
+        m="${wheel_m}" r="${wheel_r}" h="${wheel_h}"/>  <!-- Hind Right -->
 </robot>

Commit message: Added files for tutorial 3

File: src/basic_robotics/urdf/fwb_macros.xacro (robot description, xacro)
@@ -69,4 +69,10 @@
                 </geometry>
             </visual>
+            <collision>
+                <origin xyz="0.0 0.0 0.0" rpy="0.0 0.0 0.0"/>
+                <geometry>
+                    <cylinder radius="${r}" length="${h}"/>
+                </geometry>
+            </collision>
         </link>
         <!-- Joint from wheel to body -->
