Commit message: Added translation node, completing Tutorial 4

File: src/basic_robotics/urdf/fwb_gazebo_t4.urdf (robot description, URDF)
Before this commit: robot fw_robot, 5 links, 4 joints
Links:
- added link camera_link, mass 0.06; collision box size=0.015 0.045 0.06; visual box size=0.015 0.045 0.06
- added link dummy
- added link lidar_link, mass 0.12; collision box size=0.05 0.05 0.07; visual box size=0.05 0.05 0.07
Joints:
- added joint camera_joint: type fixed, parent body, child camera_link, origin xyz=0.2645 0.0 0.16
- added joint dummy_body_fixed: type fixed, parent dummy, child body, origin xyz=0.0 0.0 0.0 rpy=0.0 0.0 0.0
- added joint lidar_joint: type fixed, parent body, child lidar_link, origin xyz=0.29700000000000004 0.0 -0.095

File: src/basic_robotics/urdf/fwb_gazebo_t4.xacro (robot description, xacro)
@@ -17,4 +17,13 @@
     <xacro:include filename="$(find basic_robotics)/urdf/fwb_lidar_t4.xacro" />
     <!-- Main code -->
+    <link name="dummy">
+        <!--
+            This is a dummy link for KDL to parse the URDF. Basically, a
+            root link with <inertia> is not supported by KDL [1] (a library
+            used by robot_state_publisher). Reference at [2]
+            [1]: https://www.orocos.org/kdl.html
+            [2]: https://answers.ros.org/question/192817/error-msg-the-root-link_base-has-an-inertia-specified-in-the-urdf-but-kdl/
+        -->
+    </link>
     <!-- Main body link -->
     <link name="body">
@@ -37,4 +46,10 @@
         </collition>
     </link>
+    <!-- Attach the dummy link -->
+    <joint name="dummy_body_fixed" type="fixed">
+        <origin xyz="0.0 0.0 0.0" rpy="0.0 0.0 0.0" />
+        <parent link="dummy" />
+        <child link="body" />
+    </joint>
     <!-- Attach the wheels -->
     <xacro:add_wheel lname="fl_wheel" jname="fl_wheel_joint"
